File: 12ChannelEMG.brd (EAGLE design)
At the start: 47.4 x 269.2 mm, 89 parts

Commit message: Channel 6
Parts:
- added C29, C30, C34, C35, C36, C37, C41, C42: 0.1uF, resistor:C1206K
- added C31, C38: 3.3uF, resistor:C1206K
- added C32, C33, C39, C40: 0.22uF, rcl:C0603K
- added D5, D6: BAT54, diode:SOT23
- added R41, R51: 50k, rcl:R0805
- added R42, R50, R52, R60: 100, resistor:R0603
- added R43, R53: 10k, rcl:R0603
- added R44, R54: 200, rcl:R0603
- added R45, R46, R55, R56: 82k, resistor:R0603
- added R47, R57: 300, resistor:R0603
- added R48, R58: 100k, resistor:R0603
- added R49, R59: 56k, resistor:R0603
- added U$17, U$21: INA101KU, 12-ChannelEMG:SOIC167.5MM
- added U$18, U$22: LMC6492, 12-ChannelEMG:SOIC14
- added U$19, U$23: PV36504, 12-ChannelEMG:PV36W
- added U$20, U$24: 2PIN, 12-ChannelEMG:2PIN
Connections:
- new net N$67: R41.2, U$17.12, U$17.13
- new net N$68: U$17.3, U$20.2
- new net N$69: R42.2, U$18.2, U$19.1
- new net N$70: R42.1, U$17.1
- new net N$71: C31.1, U$18.1, U$19.2
- new net N$72: C31.2, R43.2, U$18.5
- new net N$73: R44.1, U$18.6, U$18.7
- new net N$74: R44.2, R50.1, U$18.9
- new net N$75: D5.1, U$18.8
- new net N$76: C34.1, R46.1, U$18.12
- new net N$77: D5.3, R45.1, R47.1, R50.2
- new net N$78: C35.2, R49.2, U$18.14
- new net N$79: R48.1, R49.1, U$18.13
- new net N$80: C35.1, R45.2, R46.2
- new net N$81: R41.1, U$17.4, U$17.5
- new net N$82: U$17.14, U$20.1
- new net N$83: R51.2, U$21.12, U$21.13
- new net N$84: U$21.3, U$24.2
- new net N$85: R52.2, U$22.2, U$23.1
- new net N$86: R52.1, U$21.1
- new net N$87: C38.1, U$22.1, U$23.2
- new net N$88: C38.2, R53.2, U$22.5
- new net N$89: R54.1, U$22.6, U$22.7
- new net N$90: R54.2, R60.1, U$22.9
- new net N$91: D6.1, U$22.8
- new net N$92: C41.1, R56.1, U$22.12
- new net N$93: D6.3, R55.1, R57.1, R60.2
- new net N$94: C42.2, R59.2, U$22.14
- new net N$95: R58.1, R59.1, U$22.13
- new net N$96: C42.1, R55.2, R56.2
- new net N$97: R51.1, U$21.4, U$21.5
- new net N$98: U$21.14, U$24.1
- net GND: now also C29.2, C30.2, C32.2, C33.2, C34.2, C36.2, C37.2, C39.2, C40.2, C41.2, R43.1, R47.2, R48.2, R53.1, R57.2, R58.2, U$18.10, U$18.3, U$22.10, U$22.3
- net VCC+: now also C29.1, C32.1, C36.1, C39.1, U$17.2, U$18.4, U$21.2, U$22.4
- net VCC-: now also C30.1, C33.1, C37.1, C40.1, U$17.15, U$18.11, U$21.15, U$22.11
Routing:
- net VCC-: track 182.7 -> 279.8 mm
- net VCC+: track 158.7 -> 243.4 mm, vias 11 -> 17
- net N$85: track 0.00 -> 18.0 mm, vias 0 -> 1
- net N$69: track 0.00 -> 18.0 mm, vias 0 -> 1
- net N$98: track 0.00 -> 15.9 mm, vias 0 -> 1
- net N$82: track 0.00 -> 15.9 mm, vias 0 -> 1
- net N$93: track 0.00 -> 13.4 mm, vias 0 -> 1
- net N$77: track 0.00 -> 13.4 mm, vias 0 -> 1
- net N$87: track 0.00 -> 10.1 mm
- net N$71: track 0.00 -> 10.1 mm
- net N$72: track 0.00 -> 9.66 mm
- net N$88: track 0.00 -> 9.66 mm
- net N$84: track 0.00 -> 8.31 mm
- net N$68: track 0.00 -> 8.31 mm
- net N$96: track 0.00 -> 8.14 mm
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
Commit message: Channel 9
Parts:
- added C43, C44, C48, C49, C50, C51, C55, C56, C57, C58, C62, C63: 0.1uF, resistor:C1206K
- added C45, C52, C59: 3.3uF, resistor:C1206K
- added C46, C47, C53, C54, C60, C61: 0.22uF, rcl:C0603K
- added D7, D8, D9: BAT54, diode:SOT23
- added R61, R71, R81: 50k, rcl:R0805
- added R62, R70, R72, R80, R82, R90: 100, resistor:R0603
- added R63, R73, R83: 10k, rcl:R0603
- added R64, R74, R84: 200, rcl:R0603
- added R65, R66, R75, R76, R85, R86: 82k, resistor:R0603
- added R67, R77, R87: 300, resistor:R0603
- added R68, R78, R88: 100k, resistor:R0603
- added R69, R79, R89: 56k, resistor:R0603
- added U$25, U$29, U$33: INA101KU, 12-ChannelEMG:SOIC167.5MM
- added U$26, U$30, U$34: LMC6492, 12-ChannelEMG:SOIC14
- added U$27, U$31, U$35: PV36504, 12-ChannelEMG:PV36W
- added U$28, U$32, U$36: 2PIN, 12-ChannelEMG:2PIN
Connections:
- new net N$100: U$25.3, U$28.2
- new net N$101: R62.2, U$26.2, U$27.1
- new net N$102: R62.1, U$25.1
- new net N$103: C45.1, U$26.1, U$27.2
- new net N$104: C45.2, R63.2, U$26.5
- new net N$105: R64.1, U$26.6, U$26.7
- new net N$106: R64.2, R70.1, U$26.9
- new net N$107: D7.1, U$26.8
- new net N$108: C48.1, R66.1, U$26.12
- new net N$109: D7.3, R65.1, R67.1, R70.2
- new net N$110: C49.2, R69.2, U$26.14
- new net N$111: R68.1, R69.1, U$26.13
- new net N$112: C49.1, R65.2, R66.2
- new net N$113: R61.1, U$25.4, U$25.5
- new net N$114: U$25.14, U$28.1
- new net N$115: R71.2, U$29.12, U$29.13
- new net N$116: U$29.3, U$32.2
- new net N$117: R72.2, U$30.2, U$31.1
- new net N$118: R72.1, U$29.1
- new net N$119: C52.1, U$30.1, U$31.2
- new net N$120: C52.2, R73.2, U$30.5
- new net N$121: R74.1, U$30.6, U$30.7
- new net N$122: R74.2, R80.1, U$30.9
- new net N$123: D8.1, U$30.8
- new net N$124: C55.1, R76.1, U$30.12
- new net N$125: D8.3, R75.1, R77.1, R80.2
- new net N$126: C56.2, R79.2, U$30.14
- new net N$127: R78.1, R79.1, U$30.13
- new net N$128: C56.1, R75.2, R76.2
- new net N$129: R71.1, U$29.4, U$29.5
- new net N$130: U$29.14, U$32.1
- new net N$131: R81.2, U$33.12, U$33.13
- new net N$132: U$33.3, U$36.2
- new net N$133: R82.2, U$34.2, U$35.1
- new net N$134: R82.1, U$33.1
- new net N$135: C59.1, U$34.1, U$35.2
- new net N$136: C59.2, R83.2, U$34.5
- new net N$137: R84.1, U$34.6, U$34.7
- new net N$138: R84.2, R90.1, U$34.9
- new net N$139: D9.1, U$34.8
- new net N$140: C62.1, R86.1, U$34.12
- new net N$141: D9.3, R85.1, R87.1, R90.2
- new net N$142: C63.2, R89.2, U$34.14
- new net N$143: R88.1, R89.1, U$34.13
- new net N$144: C63.1, R85.2, R86.2
- new net N$145: R81.1, U$33.4, U$33.5
- new net N$146: U$33.14, U$36.1
- new net N$99: R61.2, U$25.12, U$25.13
- net GND: now also C43.2, C44.2, C46.2, C47.2, C48.2, C50.2, C51.2, C53.2, C54.2, C55.2, C57.2, C58.2, C60.2, C61.2, C62.2, R63.1, R67.2, R68.2, R73.1, R77.2, R78.2, R83.1, R87.2, R88.2, U$26.10, U$26.3, U$30.10, U$30.3, U$34.10, U$34.3
- net VCC+: now also C43.1, C46.1, C50.1, C53.1, C57.1, C60.1, U$25.2, U$26.4, U$29.2, U$30.4, U$33.2, U$34.4
- net VCC-: now also C44.1, C47.1, C51.1, C54.1, C58.1, C61.1, U$25.15, U$26.11, U$29.15, U$30.11, U$33.15, U$34.11
Routing:
- net VCC-: track 279.8 -> 425.4 mm
- net VCC+: track 243.4 -> 370.4 mm, vias 17 -> 26
- net N$133: track 0.00 -> 18.0 mm, vias 0 -> 1
- net N$117: track 0.00 -> 18.0 mm, vias 0 -> 1
- net N$101: track 0.00 -> 18.0 mm, vias 0 -> 1
- net N$146: track 0.00 -> 15.9 mm, vias 0 -> 1
- net N$130: track 0.00 -> 15.9 mm, vias 0 -> 1
- net N$114: track 0.00 -> 15.9 mm, vias 0 -> 1
- net N$141: track 0.00 -> 13.4 mm, vias 0 -> 1
- net N$125: track 0.00 -> 13.4 mm, vias 0 -> 1
- net N$109: track 0.00 -> 13.4 mm, vias 0 -> 1
- net GND: track 24.3 -> 36.5 mm, vias 24 -> 36
- net N$135: track 0.00 -> 10.1 mm
- net N$119: track 0.00 -> 10.1 mm
- net N$103: track 0.00 -> 10.1 mm
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
Commit message: Channel 11
Parts:
- added C64, C65, C69, C70, C71, C72, C76, C77: 0.1uF, resistor:C1206K
- added C66, C73: 3.3uF, resistor:C1206K
- added C67, C68, C74, C75: 0.22uF, rcl:C0603K
- added D10, D11: BAT54, diode:SOT23
- added R100, R102, R110, R92: 100, resistor:R0603
- added R101, R91: 50k, rcl:R0805
- added R103, R93: 10k, rcl:R0603
- added R104, R94: 200, rcl:R0603
- added R105, R106, R95, R96: 82k, resistor:R0603
- added R107, R97: 300, resistor:R0603
- added R108, R98: 100k, resistor:R0603
- added R109, R99: 56k, resistor:R0603
- added U$37, U$41: INA101KU, 12-ChannelEMG:SOIC167.5MM
- added U$38, U$42: LMC6492, 12-ChannelEMG:SOIC14
- added U$39, U$43: PV36504, 12-ChannelEMG:PV36W
- added U$40, U$44: 2PIN, 12-ChannelEMG:2PIN
Connections:
- new net N$147: R91.2, U$37.12, U$37.13
- new net N$148: U$37.3, U$40.2
- new net N$149: R92.2, U$38.2, U$39.1
- new net N$150: R92.1, U$37.1
- new net N$151: C66.1, U$38.1, U$39.2
- new net N$152: C66.2, R93.2, U$38.5
- new net N$153: R94.1, U$38.6, U$38.7
- new net N$154: R100.1, R94.2, U$38.9
- new net N$155: D10.1, U$38.8
- new net N$156: C69.1, R96.1, U$38.12
- new net N$157: D10.3, R100.2, R95.1, R97.1
- new net N$158: C70.2, R99.2, U$38.14
- new net N$159: R98.1, R99.1, U$38.13
- new net N$160: C70.1, R95.2, R96.2
- new net N$161: R91.1, U$37.4, U$37.5
- new net N$162: U$37.14, U$40.1
- new net N$163: R101.2, U$41.12, U$41.13
- new net N$164: U$41.3, U$44.2
- new net N$165: R102.2, U$42.2, U$43.1
- new net N$166: R102.1, U$41.1
- new net N$167: C73.1, U$42.1, U$43.2
- new net N$168: C73.2, R103.2, U$42.5
- new net N$169: R104.1, U$42.6, U$42.7
- new net N$170: R104.2, R110.1, U$42.9
- new net N$171: D11.1, U$42.8
- new net N$172: C76.1, R106.1, U$42.12
- new net N$173: D11.3, R105.1, R107.1, R110.2
- new net N$174: C77.2, R109.2, U$42.14
- new net N$175: R108.1, R109.1, U$42.13
- new net N$176: C77.1, R105.2, R106.2
- new net N$177: R101.1, U$41.4, U$41.5
- new net N$178: U$41.14, U$44.1
- net GND: now also C64.2, C65.2, C67.2, C68.2, C69.2, C71.2, C72.2, C74.2, C75.2, C76.2, R103.1, R107.2, R108.2, R93.1, R97.2, R98.2, U$38.10, U$38.3, U$42.10, U$42.3
- net VCC+: now also C64.1, C67.1, C71.1, C74.1, U$37.2, U$38.4, U$41.2, U$42.4
- net VCC-: now also C65.1, C68.1, C72.1, C75.1, U$37.15, U$38.11, U$41.15, U$42.11
Routing:
- net VCC-: track 425.4 -> 522.5 mm
- net VCC+: track 370.4 -> 455.0 mm, vias 26 -> 32
- net N$165: track 0.00 -> 18.0 mm, vias 0 -> 1
- net N$149: track 0.00 -> 18.0 mm, vias 0 -> 1
- net N$178: track 0.00 -> 15.9 mm, vias 0 -> 1
- net N$162: track 0.00 -> 15.9 mm, vias 0 -> 1
- net N$157: track 0.00 -> 13.4 mm, vias 0 -> 1
- net N$173: track 0.00 -> 13.4 mm, vias 0 -> 1
- net N$167: track 0.00 -> 10.1 mm
- net N$151: track 0.00 -> 10.1 mm
- net N$152: track 0.00 -> 9.66 mm
- net N$168: track 0.00 -> 9.66 mm
- net N$164: track 0.00 -> 8.31 mm
- net N$148: track 0.00 -> 8.31 mm
- net N$176: track 0.00 -> 8.14 mm
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